File: ruler/ruler.kicad_pcb (KiCad board)
At the start: 2 copper layers, 32 parts, among them J1 USB_B_Micro, J2 Conn_01x05_Female, J3 Conn_01x05_Female, SW1 SW_Push_Dual, U1 SAMD21E17A, U2 AP2112K-3.3

Commit message: laid things out
Parts:
- moved TP3 57.0 mm to (117.7, 64.0)
- moved R6 55.2 mm to (185.7, 59.2), turned to 180 degrees
- moved C3 54.7 mm to (90.4, 74.7)
- moved R7 54.5 mm to (95.6, 88.4), turned to 180 degrees
- moved TP4 51.0 mm to (134.4, 64.6)
- moved C4 49.7 mm to (88.5, 83.8), turned to 180 degrees
- moved D5 47.0 mm to (185.8, 54.0)
- moved TP5 45.6 mm to (159.3, 63.2)
- moved D9 44.6 mm to (95.7, 84.8)
- moved TP6 42.3 mm to (185.1, 66.0)
- moved TP1 41.3 mm to (95.1, 106.6)
- moved TP2 41.3 mm to (103.4, 106.6)
- moved R1 40.4 mm to (192.9, 66.2), turned to 180 degrees
- moved C1 36.8 mm to (115.3, 80.6)
- moved R3 35.4 mm to (117.2, 57.3)
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